File: design/power/omi_v1_power/udimm-edge-interface.kicad_sch (KiCad schematic)
At the start: 0 parts

Commit message: feat(phase2): place J1 edge connector on the edge sheet + ERC/netlist evidence
Fills the previously-empty udimm-edge-interface.kicad_sch with one J1 instance
of omi:DDR4_UDIMM_288_Edge and a global_label (the design's dominant label type)
on every non-NC pin, so the omi_net names merge across sheets. NC pins are left
unconnected per their no_connect type. Only the edge sheet is modified.

Validated: ERC + netlist run; sheet renders. Netlist shows J1 with all 288 pins
on the expected nets (79->A0, 2->GND, 59->VDD, 3->D0_DQ4, ...); 125 nets merge
with other components; 36 NC pins add zero ERC cost.

ERC delta vs baseline: 131 -> 135 (+4) = 3 global_label_dangling
(ALERT_n/PARITY/VTT, host-side) + 1 same_local_global_label (VREF local-vs-global).
Both are Phase-3 cross-sheet reconciliation; reported here, not fixed.

Co-Authored-By: Claude Opus 4.8 (1M context) <noreply@anthropic.com>
Parts:
- added J1: DDR4_UDIMM_288_Edge, symbol omi:DDR4_UDIMM_288_Edge
Connections:
- new net A0: J1.79 (A0)
- new net A1: J1.72 (A1)
- new net A10: J1.225 (A10/AP)
- new net A11: J1.210 (A11)
- new net A12: J1.65 (A12/BC_n)
- new net A13: J1.232 (A13)
- new net A14: J1.228 (WE_n/A14)
- new net A15: J1.86 (CAS_n/A15)
- new net A16: J1.82 (RAS_n/A16)
- new net A2: J1.216 (A2)
- new net A3: J1.71 (A3)
- new net A4: J1.214 (A4)
- new net A5: J1.213 (A5)
- new net A6: J1.69 (A6)
- new net A7: J1.211 (A7)
- new net A8: J1.68 (A8)
- new net A9: J1.66 (A9)
- new net ACT_n: J1.62 (ACT_n)
- new net ALERT_n: J1.208 (ALERT_n)
- new net BA0: J1.81 (BA0)
- new net BA1: J1.224 (BA1)
- new net BG0: J1.63 (BG0)
- new net BG1: J1.207 (BG1)
- new net CKE0: J1.60 (CKE0)
- new net CK_c: J1.75 (CK0_c)
- new net CK_t: J1.74 (CK0_t)
- new net CS0_n: J1.84 (CS0_n)
- new net D0_DM_DBI_n: J1.7 (DM0_n/DBI0_n)
- new net D0_DQ0: J1.5 (DQ0)
- new net D0_DQ1: J1.150 (DQ1)
- new net D0_DQ2: J1.12 (DQ2)
- new net D0_DQ3: J1.157 (DQ3)
- new net D0_DQ4: J1.3 (DQ4)
- new net D0_DQ5: J1.148 (DQ5)
- new net D0_DQ6: J1.10 (DQ6)
- new net D0_DQ7: J1.155 (DQ7)
- new net D0_DQS_c: J1.152 (DQS0_c)
- new net D0_DQS_t: J1.153 (DQS0_t)
- new net D1_DM_DBI_n: J1.18 (DM1_n/DBI1_n)
- new net D1_DQ0: J1.16 (DQ8)
- new net D1_DQ1: J1.161 (DQ9)
- new net D1_DQ2: J1.23 (DQ10)
- new net D1_DQ3: J1.168 (DQ11)
- new net D1_DQ4: J1.14 (DQ12)
- new net D1_DQ5: J1.159 (DQ13)
- new net D1_DQ6: J1.21 (DQ14)
- new net D1_DQ7: J1.166 (DQ15)
- new net D1_DQS_c: J1.163 (DQS1_c)
- new net D1_DQS_t: J1.164 (DQS1_t)
- new net D2_DM_DBI_n: J1.29 (DM2_n/DBI2_n)
- new net D2_DQ0: J1.27 (DQ16)
- new net D2_DQ1: J1.172 (DQ17)
- new net D2_DQ2: J1.34 (DQ18)
- new net D2_DQ3: J1.179 (DQ19)
- new net D2_DQ4: J1.25 (DQ20)
- new net D2_DQ5: J1.170 (DQ21)
- new net D2_DQ6: J1.32 (DQ22)
- new net D2_DQ7: J1.177 (DQ23)
- new net D2_DQS_c: J1.174 (DQS2_c)
- new net D2_DQS_t: J1.175 (DQS2_t)
- new net D3_DM_DBI_n: J1.40 (DM3_n/DBI3_n)
- new net D3_DQ0: J1.38 (DQ24)
- new net D3_DQ1: J1.183 (DQ25)
- new net D3_DQ2: J1.45 (DQ26)
- new net D3_DQ3: J1.190 (DQ27)
- new net D3_DQ4: J1.36 (DQ28)
- new net D3_DQ5: J1.181 (DQ29)
- new net D3_DQ6: J1.43 (DQ30)
- new net D3_DQ7: J1.188 (DQ31)
- new net D3_DQS_c: J1.185 (DQS3_c)
- new net D3_DQS_t: J1.186 (DQS3_t)
- new net D4_DM_DBI_n: J1.99 (DM4_n/DBI4_n)
- new net D4_DQ0: J1.97 (DQ32)
- new net D4_DQ1: J1.242 (DQ33)
- new net D4_DQ2: J1.104 (DQ34)
- new net D4_DQ3: J1.249 (DQ35)
- new net D4_DQ4: J1.95 (DQ36)
- new net D4_DQ5: J1.240 (DQ37)
- new net D4_DQ6: J1.102 (DQ38)
- new net D4_DQ7: J1.247 (DQ39)
- new net D4_DQS_c: J1.244 (DQS4_c)
- new net D4_DQS_t: J1.245 (DQS4_t)
- new net D5_DM_DBI_n: J1.110 (DM5_n/DBI5_n)
- new net D5_DQ0: J1.108 (DQ40)
- new net D5_DQ1: J1.253 (DQ41)
- new net D5_DQ2: J1.115 (DQ42)
- new net D5_DQ3: J1.260 (DQ43)
- new net D5_DQ4: J1.106 (DQ44)
- new net D5_DQ5: J1.251 (DQ45)
- new net D5_DQ6: J1.113 (DQ46)
- new net D5_DQ7: J1.258 (DQ47)
- new net D5_DQS_c: J1.255 (DQS5_c)
- new net D5_DQS_t: J1.256 (DQS5_t)
- new net D6_DM_DBI_n: J1.121 (DM6_n/DBI6_n)
- new net D6_DQ0: J1.119 (DQ48)
- new net D6_DQ1: J1.264 (DQ49)
- new net D6_DQ2: J1.126 (DQ50)
- new net D6_DQ3: J1.271 (DQ51)
- new net D6_DQ4: J1.117 (DQ52)
- new net D6_DQ5: J1.262 (DQ53)
- new net D6_DQ6: J1.124 (DQ54)
- new net D6_DQ7: J1.269 (DQ55)
- new net D6_DQS_c: J1.266 (DQS6_c)
- new net D6_DQS_t: J1.267 (DQS6_t)
- new net D7_DM_DBI_n: J1.132 (DM7_n/DBI7_n)
- new net D7_DQ0: J1.130 (DQ56)
- new net D7_DQ1: J1.275 (DQ57)
- new net D7_DQ2: J1.137 (DQ58)
- new net D7_DQ3: J1.282 (DQ59)
- new net D7_DQ4: J1.128 (DQ60)
- new net D7_DQ5: J1.273 (DQ61)
- new net D7_DQ6: J1.135 (DQ62)
- new net D7_DQ7: J1.280 (DQ63)
- new net D7_DQS_c: J1.277 (DQS7_c)
- new net D7_DQS_t: J1.278 (DQS7_t)
- new net GND: J1.101 (VSS), J1.103 (VSS), J1.105 (VSS), J1.107 (VSS), J1.109 (VSS), J1.11 (VSS), J1.112 (VSS), J1.114 (VSS), J1.116 (VSS), J1.118 (VSS), J1.120 (VSS), J1.123 (VSS), J1.125 (VSS), J1.127 (VSS), J1.129 (VSS), J1.13 (VSS), J1.131 (VSS), J1.134 (VSS), J1.136 (VSS), J1.138 (VSS), J1.147 (VSS), J1.149 (VSS), J1.15 (VSS), J1.151 (VSS), J1.154 (VSS), J1.156 (VSS), J1.158 (VSS), J1.160 (VSS), J1.162 (VSS), J1.165 (VSS), J1.167 (VSS), J1.169 (VSS), J1.17 (VSS), J1.171 (VSS), J1.173 (VSS), J1.176 (VSS), J1.178 (VSS), J1.180 (VSS), J1.182 (VSS), J1.184 (VSS), J1.187 (VSS), J1.189 (VSS), J1.191 (VSS), J1.193 (VSS), J1.195 (VSS), J1.198 (VSS), J1.2 (VSS), J1.20 (VSS), J1.200 (VSS), J1.202 (VSS), J1.22 (VSS), J1.24 (VSS), J1.241 (VSS), J1.243 (VSS), J1.246 (VSS), J1.248 (VSS), J1.250 (VSS), J1.252 (VSS), J1.254 (VSS), J1.257 (VSS), J1.259 (VSS), J1.26 (VSS), J1.261 (VSS), J1.263 (VSS), J1.265 (VSS), J1.268 (VSS), J1.270 (VSS), J1.272 (VSS), J1.274 (VSS), J1.276 (VSS), J1.279 (VSS), J1.28 (VSS), J1.281 (VSS), J1.283 (VSS), J1.31 (VSS), J1.33 (VSS), J1.35 (VSS), J1.37 (VSS), J1.39 (VSS), J1.4 (VSS), J1.42 (VSS), J1.44 (VSS), J1.46 (VSS), J1.48 (VSS), J1.50 (VSS), J1.53 (VSS), J1.55 (VSS), J1.57 (VSS), J1.6 (VSS), J1.9 (VSS), J1.94 (VSS), J1.96 (VSS), J1.98 (VSS)
- new net ODT0: J1.87 (ODT0)
- new net PARITY: J1.222 (PARITY)
- new net RESET_n: J1.58 (RESET_n)
- new net SA0: J1.139 (SA0)
- new net SA1: J1.140 (SA1)
- new net SA2: J1.238 (SA2)
- new net SPD_SCL: J1.141 (SCL)
- new net SPD_SDA: J1.285 (SDA)
- new net VDD: J1.204 (VDD), J1.206 (VDD), J1.209 (VDD), J1.212 (VDD), J1.215 (VDD), J1.217 (VDD), J1.220 (VDD), J1.223 (VDD), J1.226 (VDD), J1.229 (VDD), J1.231 (VDD), J1.233 (VDD), J1.236 (VDD), J1.239 (VDD), J1.59 (VDD), J1.61 (VDD), J1.64 (VDD), J1.67 (VDD), J1.70 (VDD), J1.73 (VDD), J1.76 (VDD), J1.80 (VDD), J1.83 (VDD), J1.85 (VDD), J1.88 (VDD), J1.90 (VDD), J1.92 (VDD)
- new net VDDSPD: J1.284 (VDDSPD)
- new net VPP: J1.142 (VPP), J1.143 (VPP), J1.286 (VPP), J1.287 (VPP), J1.288 (VPP)
- new net VREF: J1.146 (VREFCA)
- new net VTT: J1.221 (VTT), J1.77 (VTT)
