File: design/power/omi_v1_power/udimm-edge-interface.kicad_sch (KiCad schematic)
At the start: 1 part, among them J1 DDR4_UDIMM_288_Edge

Commit message: feat(phase4): assign J1 card-edge footprint on the schematic instance
Set the Footprint property on the placed J1 symbol (edge sheet) to
omi:DDR4_UDIMM_288_Edge (NOT in omi.kicad_sym -> symbol stays frozen). Validated:
netlist shows footprints for all 10 real components (J1 + U_DRAM0-7 + U_SPD0);
power symbols correctly carry none; J1 footprint pads {1..288} == symbol pins
{1..288} (sets exactly equal); ERC unchanged at 85; omi.kicad_sym +
tools/edge_symbol untouched. DRAM (FBGA-78) + SPD (DFN-8) confirmed correct,
no change needed.

Co-Authored-By: Claude Opus 4.8 (1M context) <noreply@anthropic.com>
Parts:
- J1: footprint (none) -> omi:DDR4_UDIMM_288_Edge
Changed lines of the file:
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@@
 			)
 		)
-		(property "Footprint" ""
+		(property "Footprint" "omi:DDR4_UDIMM_288_Edge"
 			(at 152.4 190.5 0)
 			(effects

Commit message: polish(schematic): v1.1.0 title blocks + sheet annotations (no electrical change)
Hand-done KiCad 9 GUI pass over all five schematic sheets. Title-block
and text-box content only — no wiring, no component, no net changes.

- Title block (all sheets): Company=OMI, Rev=1.1.0, Date=2026-06-02,
  plus functional per-sheet titles.
- Repurposed the previously-empty DQ/DQS sheet into a byte-lane reference table.
- Added a mechanical caveat text box on the edge (UDIMM) sheet.
- Added a power-rail summary text box on the root sheet.
- omi_v1_power.kicad_prl: project-local UI state saved with the GUI session.

Electrical integrity is asserted to be unchanged and is verified downstream
by the export pipeline (ERC=0 gate + byte-identical netlist and BOM).

Co-Authored-By: Claude Opus 4.8 (1M context) <noreply@anthropic.com>
Other:
- note added: "UDIMM 288-Pin Edge Interface J1 - DDR4 UDIMM 288-pin card edge. Pin assignment per ddr4_udimm_288_pinmap.csv (keystone source of truth). Mechanical outline, Edge.Cuts, and JEDEC key-notch position are NOT defined in v1. Footprint is pads-only and NOT JEDEC-mechanically verified - not fab-ready."
- company: (none) -> OMI
- title: (none) -> UDIMM 288-Pin Edge Interface
- moved on the sheet: J1
